File: KiCad/ModulinV2/ModulinV2.kicad_pcb (KiCad board)
At the start: 4 copper layers, 652 parts, among them IC1 TL074HIDR, IC10 ADS7866IDBVT, IC11 DAC60501ZDGSR, IC12 DAC60501ZDGSR, IC13 AS3340D, IC14 AS3340D, IC15 TL074HIDR, IC16 TL074HIDR, IC17 TL072HIDR, IC18 SN74LV10ADR, IC19 SN74LV10ADR, IC2 STM32F401RET6, IC20 SN74LV10ADR, IC21 SN74HC193DR, IC22 TMUX4051DYYRQ1, IC23 TL072HIDR, IC24 NC7SZ74K8X, IC25 SN74AHCT1G00DBVR, IC26 SN74AHCT1G00DBVR, IC27 SN74AHCT1G00DBVR, IC28 SN74AHC1G02DBVR, IC29 SN74AHC1G02DBVR, IC3 USBLC6-2SC6, IC30 SN74HC193DR, IC31 TMUX4052DYYR, IC32 TMUX4051DYYRQ1, IC33 TMUX4051DYYRQ1, IC34 E-ULN2003D1013TR, IC35 E-ULN2003D1013TR, IC36 CD4028BM96, IC37 CD4028BM96, IC38 TL072HIDR, IC39 AS3360D, IC4 TL072HIDR, IC40 REF196GSZ-REEL, IC41 NCP5500DADJR2G, IC42 LM2576S-12_NOPB, IC43 LM2576S-12_NOPB, IC44 REF195ESZ-REEL, IC45 NCP5500DADJR2G, IC46 L7812CD2T-TR, IC47 L7812CD2T-TR, IC48 TL074HIDR, IC49 AS3310D, IC5 TL072HIDR, IC50 AS3310D, IC51 TL074HIDR, IC52 DAC53202RTER, IC53 TL072HIDR, IC54 AS3320D, IC55 TL072HIDR, IC56 AS3320D, IC6 TL074HIDR, IC7 ADS7041IDCUR, IC8 ADS7041IDCUR, IC9 ADS7866IDBVT, J1 NRJ4HF-1, J2 USB4105-GF-A, J3 TSM-103-01-T-DV, J4 TSW-104-07-G-S, J5 TSW-104-07-T-D, J6 TSW-104-07-T-D, J7 TSW-104-07-T-D, J8 TSW-104-07-T-D, J9 PJ-002B, Q1 MMBFJ201, Q2 MMBFJ201, Q3 DMP610DL-7, SW1 SW_SPDT_MSM, SW2 Rocker Switch, U1 SN74AHC1G08DBVR, Y1 CX2016FB24000B0FZZH1

Commit message: Decided to make everything one sided and not care about layout as much
Parts:
- C140, C19, C22, C24, C27, C30, C33, C35, C37, IC43, IC47, IC5, IC6, L2, L4, R21, R22, R23, R24, R25, R29, R30, R31, R32, R33, RV2, RV3: moved to F.Cu
- TP29: moved to B.Cu
- moved C139 62.6 mm to (28.5, 71.0), turned to 180 degrees
- moved C137 58.1 mm to (21.5, 64.5), turned to -90 degrees
- moved TP67 56.1 mm to (21.5, 57.5)
- moved TP26 54.5 mm to (261.0, 105.2)
- moved C31 50.2 mm to (256.1, 93.5), turned to 0 degrees
- moved C130 48.6 mm to (75.5, 22.0), turned to 90 degrees
- moved C23 47.8 mm to (268.2, 103.0), turned to 180 degrees
- moved IC3 47.7 mm to (37.0, 137.1)
- moved R5 47.7 mm to (30.5, 141.1)
- moved R6 47.7 mm to (33.0, 138.6)
- moved RV17 47.7 mm to (33.5, 129.7)
- moved C10 47.7 mm to (61.6, 134.5)
- moved C11 47.7 mm to (55.1, 131.3)
- moved C12 47.7 mm to (55.1, 128.3)
- moved C13 47.7 mm to (55.1, 137.3)
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Routing:
- net +12V: track 114.8 -> 65.4 mm, vias 1 -> 2
- net /ADSR/GATE2: track 41.8 -> 4.35 mm
- net /PRESSURE2: track 31.9 -> 1.27 mm
- net /PRESSURE1: track 35.6 -> 5.73 mm
- net -12V: track 92.4 -> 65.5 mm, vias 2 -> 1
- net +3.3VA: track 46.7 -> 22.9 mm
- net Net-(IC6D--): track 3.82 -> 24.8 mm
- net /Interface/ADC_MISO: track 9.52 -> 28.4 mm, vias 0 -> 4
- net GND: track 10.8 -> 28.1 mm, vias 3 -> 8
- net /Interface/ADC_CLK: track 7.51 -> 24.1 mm, vias 0 -> 3
- net /ADSR/GATE1: track 30.8 -> 15.1 mm
- net Net-(D7-A): track 53.1 -> 68.8 mm
- net Net-(IC5B--): track 41.7 -> 27.0 mm
- net VDC: track 144.6 -> 132.2 mm
- net Net-(IC4A-+): track 17.1 -> 10.9 mm
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- added copper zone on In2.Cu, net +12V
- added copper zone on In2.Cu, net -12V

Commit message: Continued designing the MCU schematic
Parts:
- C10, C11, C12, C13, C14, C15, C16, C17, C18, C7, C8, C9, IC41, R112: moved to F.Cu
- moved S3 150.8 mm to (20.8, 125.8), turned to 180 degrees
- moved R12 148.3 mm to (28.0, 126.0), turned to 90 degrees
- moved S1 142.3 mm to (28.5, 106.5), turned to 180 degrees
- moved C2 134.6 mm to (35.2, 106.5), turned to 90 degrees
- moved Y1 104.9 mm to (44.2, 121.2), turned to -90 degrees
- moved C4 103.4 mm to (40.2, 121.2), turned to -90 degrees
- moved C5 94.5 mm to (49.2, 123.0)
- moved LED1 79.5 mm to (66.9, 116.7), turned to 90 degrees
- moved R16 70.4 mm to (72.1, 121.2), turned to 180 degrees
- moved R15 70.3 mm to (72.1, 118.2)
- moved R17 69.4 mm to (72.1, 115.2)
- moved LED19 61.9 mm to (48.8, 89.2), turned to 180 degrees
- moved R117 58.1 mm to (42.2, 89.2), turned to 0 degrees
- moved R112 57.9 mm to (43.0, 84.5)
- moved IC41 57.2 mm to (40.2, 79.2), turned to 0 degrees
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Connections:
- IC2 pad 29: /MCU/LED_B -> unconnected-(IC2-PB10-Pad29)
- IC2 pad 57: unconnected-(IC2-PB5-Pad57) -> /MCU/LED_B
Routing:
- net /MCU/USB_D-: track 0.00 -> 17.8 mm
- net /MCU/USB_D+: track 0.00 -> 17.6 mm
- net GND: track 28.1 -> 45.6 mm
- net +5V: track 36.9 -> 54.1 mm, vias 1 -> 0
- net Net-(IC5B--): track 27.0 -> 41.4 mm
- net /MCU/OSC2: track 0.00 -> 13.3 mm
- net /PRESSURE2: track 1.27 -> 14.5 mm, vias 2 -> 0
- net /MCU/OSC1: track 0.00 -> 11.6 mm
- net /MCU/NRST: track 0.00 -> 10.7 mm, vias 0 -> 2
- net /ADSR/GATE2: track 4.35 -> 14.1 mm
- net Net-(LED1-Pad3): track 0.00 -> 9.12 mm
- net Net-(LED1-Pad2): track 0.00 -> 5.46 mm
- net /MCU/BOOT: track 0.00 -> 4.57 mm
- net Net-(IC45-ADJ): track 13.4 -> 9.11 mm
- net Net-(LED1-Pad4): track 0.00 -> 3.99 mm
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